Commit message: DID ALOT OF STUFF: - Restructured models directory - Added more maps - Added directory for datasets and perspectives (rqt views) - New scripts for running different things - Added a lot of documentation - Split up follow_uav into multiple files and added a lot of functionality to it - Now follow_uav is basically just leader estimater and controller, with the rest of the functionality split up into separate files - follow_uav_odom is a new node that is basically the same as follow_uav but it uses odometry instead of camera tracking for the follower pose estimation, and it is used for debugging and testing the controller without the camera tracking in the loop - The math and debug files are for testing and debugging the follow_uav functionality, and they are not used in the main follow_uav node, but they are used in the run_follow_yaw_debug.py script for testing the yaw control of the follower - Implemented Nav2 as a ugv_mode - Added some scanned maps, but only warehouse works well, the others are pretty bad and not really usable, but they are there for testing and future work - Some older stuff might be broken now (like old run scripts) - We also spawn the UAV with camera attached as default again, detached introduced lags and delays
See RUNNING_SIM.md for instructions on how to run the new stuff, and the new README.md for an overview of the project and the new structure.

File: src/lrs_halmstad/clearpath/robot.urdf.xacro (robot description, xacro)
@@ -22,9 +22,9 @@
   <!-- Mounts -->
   <!-- Sensors -->
-  <!-- lidar3d_0 -->
-  <xacro:include filename="$(find clearpath_sensors_description)/urdf/velodyne_lidar.urdf.xacro"/>
-  <xacro:velodyne_lidar name="lidar3d_0" parent_link="base_link" ang_res_h="0.4" ang_res_v="2.0" min_ang_h="-3.141592" max_ang_h="3.141592" min_ang_v="-0.261799" max_ang_v="0.261799" min_range="0.9" max_range="130.0" update_rate="20">
+  <!-- lidar2d_0 -->
+  <xacro:include filename="$(find clearpath_sensors_description)/urdf/hokuyo_ust.urdf.xacro"/>
+  <xacro:hokuyo_ust name="lidar2d_0" parent_link="base_link" ang_res="0.5" min_ang="-3.141592653589793" max_ang="3.141592653589793" min_range="0.05" max_range="25.0" update_rate="40">
     <origin xyz="0.21 0.13 0.225" rpy="0.0 0.0 0.0"/>
-  </xacro:velodyne_lidar>
+  </xacro:hokuyo_ust>
   <!-- camera_0 -->
   <xacro:include filename="$(find clearpath_sensors_description)/urdf/intel_realsense.urdf.xacro"/>

File: src/lrs_halmstad/xacro/lrs_camera_gimbal.sdf.xacro (robot description, xacro)
@@ -3,15 +3,33 @@
     <xacro:property name="M_PI" value="3.1415926535897931"/>
     <xacro:macro name="lrs_camera_gimbal"
-                 params="name parent_link link_name image_topic camera_info_topic frame_id update_rate im_width im_height im_format hfov_deg far_clip robot_type robot_name x_offset:=0.0 y_offset:=0.0 z_offset:=0.0 pitch_offset:=0.0 yaw_offset:=0.0">
+                 params="name parent_link link_name image_topic camera_info_topic frame_id update_rate im_width im_height im_format hfov_deg far_clip robot_type robot_name x_offset:=0.0 y_offset:=0.0 z_offset:=0.0 pitch_offset:=0.0 yaw_offset:=0.0 sensor_roll_offset:=0.0 sensor_pitch_offset:=0.0 sensor_yaw_offset:=0.0">
       <link name="${link_name}">
          <pose rotation_format="euler_rpy" degrees="true">${x_offset} ${y_offset} ${z_offset} 0 ${pitch_offset} ${yaw_offset}</pose>
+            <gravity>false</gravity>
+            <kinematic>true</kinematic>
+            <inertial>
+                <mass>0.01</mass>
+                <inertia>
+                    <ixx>1.0e-4</ixx>
+                    <ixy>0.0</ixy>
+                    <ixz>0.0</ixz>
+                    <iyy>1.0e-4</iyy>
+                    <iyz>0.0</iyz>
+                    <izz>1.0e-4</izz>
+                </inertia>
+            </inertial>
             <visual name="visual">
-                <origin xyz="0 0 0.0" rpy="0 0 0"/>
+                <pose>0 0 0 0 0 0</pose>
                 <geometry>
 	          <mesh>
-                    <uri>model://zenmuse_z3/meshes/zenmuse_z3.dae</uri>
+                    <uri>model://zenmuse_z3/meshes/zenmuse_z3.stl</uri>
                     <scale>1.0 1.0 1.0</scale>
                   </mesh>
                 </geometry>
+                <material>
+                    <ambient>0.25 0.25 0.25 1.0</ambient>
+                    <diffuse>0.45 0.45 0.45 1.0</diffuse>
+                    <specular>0.05 0.05 0.05 1.0</specular>
+                </material>
             </visual>
             <!-- collision name="collision">
@@ -38,5 +56,5 @@
                     <!-- <pose>0.027 0 -0.027 0 1.57 0</pose> -->
                     <!-- <pose>0.027 0 -0.027 0 1.57 0</pose> -->
-                    <pose>0.027 0 -0.027 0 0 0</pose>
+                    <pose rotation_format="euler_rpy" degrees="true">0.027 0 -0.027 ${sensor_roll_offset} ${sensor_pitch_offset} ${sensor_yaw_offset}</pose>
                     <horizontal_fov>${hfov_deg * M_PI/180.0}</horizontal_fov>
                     <image>
@@ -54,5 +72,4 @@
                 <visualize>true</visualize>
                 <topic>${image_topic}</topic>
-                <ignition_frame_id>${frame_id}</ignition_frame_id>
             </sensor>
         </link>

File: src/lrs_halmstad/xacro/lrs_gimbal.xacro (robot description, xacro)
@@ -4,6 +4,7 @@
   <xacro:arg name="robot_name" default="dji0"/>
   <xacro:arg name="robot_type" default="laser"/>
+  <xacro:arg name="model_static" default="false"/>
   <model name="$(arg robot_name)_$(arg camera_name)">
-    <static>true</static>
+    <static>$(arg model_static)</static>
     <xacro:arg name="base_link_frame" default="base_link"/>
     <xacro:arg name="world_frame" default="world"/>
@@ -11,8 +12,11 @@
     <xacro:arg name="camera_image_width" default="1024"/>
     <xacro:arg name="camera_image_height" default="600"/>
-    <xacro:arg name="camera_update_rate" default="30"/>
-    <xacro:arg name="camera_hfov" default="71"/>
-    <xacro:arg name="camera_far_clip" default="100"/>
-    <xacro:arg name="camera_topic" default="image_raw"/>
+  <xacro:arg name="camera_update_rate" default="30"/>
+  <xacro:arg name="camera_hfov" default="94"/>
+  <xacro:arg name="camera_far_clip" default="100"/>
+  <xacro:arg name="camera_topic" default="image_raw"/>
+  <xacro:arg name="camera_sensor_roll_deg" default="0.0"/>
+  <xacro:arg name="camera_sensor_pitch_deg" default="0.0"/>
+  <xacro:arg name="camera_sensor_yaw_deg" default="0.0"/>
     <xacro:property name="prop_type" value="$(arg robot_type)"/>
     <xacro:property name="base_name" value="$(arg robot_name)"/>
@@ -34,4 +38,7 @@
                              robot_type="$(arg robot_type)"
                              robot_name="$(arg robot_name)"
+                             sensor_roll_offset="$(arg camera_sensor_roll_deg)"
+                             sensor_pitch_offset="$(arg camera_sensor_pitch_deg)"
+                             sensor_yaw_offset="$(arg camera_sensor_yaw_deg)"
                              im_format="R8G8B8" />
 </model>

File: src/lrs_halmstad/xacro/lrs_m100_base.sdf.xacro (robot description, xacro)
@@ -8,5 +8,5 @@
              <pose rotation_format="euler_rpy" degrees="true">0 0 0 0 0 0</pose>
             <visual name="visual">
-                <origin xyz="0 0 0" rpy="0 0 0"/>
+                <pose>0 0 0 0 0 0</pose>
                 <geometry>
 	          <mesh>
@@ -17,5 +17,5 @@
             </visual>
             <collision name="collision">
-                <origin xyz="0 0 0" rpy="0 0 0"/>
+                <pose>0 0 0 0 0 0</pose>
                 <geometry>
 	          <mesh>
