Commit message: Depth camera added

File: src/lrs_halmstad/xacro/lrs_camera_gimbal.sdf.xacro (robot description, xacro)
@@ -3,5 +3,5 @@
     <xacro:property name="M_PI" value="3.1415926535897931"/>
     <xacro:macro name="lrs_camera_gimbal"
-                 params="name parent_link link_name image_topic camera_info_topic frame_id update_rate im_width im_height im_format hfov_deg far_clip robot_type robot_name x_offset:=0.0 y_offset:=0.0 z_offset:=0.0 pitch_offset:=0.0 yaw_offset:=0.0 sensor_roll_offset:=0.0 sensor_pitch_offset:=0.0 sensor_yaw_offset:=0.0">
+                 params="name parent_link link_name topic_base frame_id update_rate im_width im_height im_format hfov_deg far_clip robot_type robot_name x_offset:=0.0 y_offset:=0.0 z_offset:=0.0 pitch_offset:=0.0 yaw_offset:=0.0 sensor_roll_offset:=0.0 sensor_pitch_offset:=0.0 sensor_yaw_offset:=0.0">
       <link name="${link_name}">
          <pose rotation_format="euler_rpy" degrees="true">${x_offset} ${y_offset} ${z_offset} 0 ${pitch_offset} ${yaw_offset}</pose>
@@ -52,5 +52,5 @@
             <child link="camera_optical_frame"/>
         </joint -->
-            <sensor type="camera" name="${robot_name}_camera_sensor">
+            <sensor type="rgbd_camera" name="${robot_name}_camera_sensor">
                 <camera>
                     <!-- <pose>0.027 0 -0.027 0 1.57 0</pose> -->
@@ -67,9 +67,11 @@
                         <far>${far_clip}</far>
                     </clip>
+                    <optical_frame_id>${frame_id}</optical_frame_id>
                 </camera>
                 <update_rate>${update_rate}</update_rate>
                 <always_on>1</always_on>
                 <visualize>true</visualize>
-                <topic>${image_topic}</topic>
+                <gz_frame_id>${frame_id}</gz_frame_id>
+                <topic>${topic_base}</topic>
             </sensor>
         </link>

File: src/lrs_halmstad/xacro/lrs_gimbal.xacro (robot description, xacro)
@@ -15,5 +15,4 @@
   <xacro:arg name="camera_hfov" default="94"/>
   <xacro:arg name="camera_far_clip" default="100"/>
-  <xacro:arg name="camera_topic" default="image_raw"/>
   <xacro:arg name="camera_sensor_roll_deg" default="0.0"/>
   <xacro:arg name="camera_sensor_pitch_deg" default="0.0"/>
@@ -22,5 +21,4 @@
     <xacro:property name="base_name" value="$(arg robot_name)"/>
     <xacro:property name="camera_prefix" value="/${base_name}/$(arg camera_name)"/>
-    <xacro:property name="camera_topic" value="$(arg camera_topic)"/>
     <xacro:property name="camera_link_name" value="$(arg camera_name)_link"/>
     <xacro:include filename="$(find lrs_halmstad)/xacro/lrs_camera_gimbal.sdf.xacro"/>
@@ -29,6 +27,5 @@
                              link_name="${camera_link_name}"
                              hfov_deg="$(arg camera_hfov)"
-                             camera_info_topic="${camera_prefix}/camera_info"
-                             image_topic="${camera_prefix}/${camera_topic}"
+                             topic_base="${camera_prefix}"
                              frame_id="${camera_prefix}/image_frame"
                              im_width="$(arg camera_image_width)"

File: src/lrs_halmstad/xacro/lrs_model.xacro (robot description, xacro)
@@ -49,5 +49,4 @@
     <xacro:arg name="camera_hfov" default="94"/>
     <xacro:arg name="camera_far_clip" default="100"/>
-    <xacro:arg name="camera_topic" default="image_raw"/>
     <xacro:arg name="camera_pitch_offset" default="+60.0"/>
     <xacro:property name="prop_type" value="$(arg robot_type)"/>
@@ -88,5 +87,4 @@
     <xacro:if value="$(arg with_camera)">
         <xacro:property name="camera_prefix" value="/${base_name}/$(arg camera_name)"/>
-        <xacro:property name="camera_topic" value="$(arg camera_topic)"/>
         <xacro:property name="camera_link_name" value="$(arg camera_name)_link"/>
         <xacro:include filename="$(find lrs_halmstad)/xacro/lrs_camera_gimbal.sdf.xacro"/>
@@ -95,6 +93,5 @@
                                  link_name="${camera_link_name}"
                                  hfov_deg="$(arg camera_hfov)"
-                                 camera_info_topic="${camera_prefix}/camera_info"
-                                 image_topic="${camera_prefix}/${camera_topic}"
+                                 topic_base="${camera_prefix}"
                                  frame_id="${camera_prefix}/image_frame"
                                  im_width="$(arg camera_image_width)"
